File: aqua-flower_hw/aqua-flower.sch (KiCad schematic (older format))
At the start: 40 parts, among them Q1 NPN, Q2 IRLML6302, Q3 IRLML6302, Q4 IRLML6302, Q5 IRLML6302, SW1 BUTTON, SW2 BUTTON, SW3 BUTTON, SW4 BUTTON, SW5 BUTTON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

Commit message: Reset Library Component
Parts:
- added HOLE1, HOLE2, HOLE3, HOLE4: HOLE_METALLED, PCB:Hole3_5_out6mm, symbol HOLE_METALLED
- DA1: footprint TO_SOT_Packages_SMD:SOT-223 -> (none)
Connections:
- wire segments 154 -> 159
Changed lines of the file:
@@
 EESchema Schematic File Version 2
+LIBS:aqua-flower-rescue
 LIBS:Connectors_kl
 LIBS:display_kl
@@
 $EndComp
 NoConn ~ 1300 1350
-$Comp
-L LD1117 DA1
-U 1 1 56FFE18D
-P 3250 1200
-F 0 "DA1" H 3150 1500 60  0000 C CNN
-F 1 "LD1117" H 3250 1400 60  0000 C CNN
-F 2 "TO_SOT_Packages_SMD:SOT-223" H 3250 1200 60  0001 C CNN
-F 3 "" H 3250 1200 60  0000 C CNN
-	1    3250 1200
-	1    0    0    -1
-$EndComp
 Wire Wire Line
 	2600 1150 2950 1150
@@
 Wire Wire Line
 	14450 5200 15100 5200
+$Comp
+L LD1117 DA1
+U 1 1 5700E1E0
+P 3250 1200
+F 0 "DA1" H 3150 1500 60  0000 C CNN
+F 1 "LD1117" H 3250 1400 60  0000 C CNN
+F 2 "" H 3250 1200 60  0001 C CNN
+F 3 "" H 3250 1200 60  0000 C CNN
+	1    3250 1200
+	1    0    0    -1
+$EndComp
+$Comp
+L HOLE_METALLED HOLE1
+U 1 1 5700EC49
+P 15050 7000
+F 0 "HOLE1" H 14550 6950 60  0000 C CNN
+F 1 "HOLE_METALLED" H 14500 7050 60  0000 C CNN
+F 2 "PCB:Hole3_5_out6mm" H 15050 7000 60  0001 C CNN
+F 3 "" H 15050 7000 60  0000 C CNN
+	1    15050 7000
+	-1   0    0    1
+$EndComp
+$Comp
+L HOLE_METALLED HOLE2
+U 1 1 5700F195
+P 15050 7250
+F 0 "HOLE2" H 14550 7200 60  0000 C CNN
+F 1 "HOLE_METALLED" H 14500 7300 60  0000 C CNN
+F 2 "PCB:Hole3_5_out6mm" H 15050 7250 60  0001 C CNN
+F 3 "" H 15050 7250 60  0000 C CNN
+	1    15050 7250
+	-1   0    0    1
+$EndComp
+$Comp
+L HOLE_METALLED HOLE3
+U 1 1 5700F547
+P 15050 7500
+F 0 "HOLE3" H 14550 7450 60  0000 C CNN
+F 1 "HOLE_METALLED" H 14500 7550 60  0000 C CNN
+F 2 "PCB:Hole3_5_out6mm" H 15050 7500 60  0001 C CNN
+F 3 "" H 15050 7500 60  0000 C CNN
+	1    15050 7500
+	-1   0    0    1
+$EndComp
+$Comp
+L HOLE_METALLED HOLE4
+U 1 1 5700F5DE
+P 15050 7750
+F 0 "HOLE4" H 14550 7700 60  0000 C CNN
+F 1 "HOLE_METALLED" H 14500 7800 60  0000 C CNN
+F 2 "PCB:Hole3_5_out6mm" H 15050 7750 60  0001 C CNN
+F 3 "" H 15050 7750 60  0000 C CNN
+	1    15050 7750
+	-1   0    0    1
+$EndComp
+Wire Wire Line
+	14750 7000 14450 7000
+Wire Wire Line
+	14450 7000 14450 7950
+Wire Wire Line
+	14750 7250 14450 7250
+Connection ~ 14450 7250
+Wire Wire Line
+	14450 7500 14750 7500
+Connection ~ 14450 7500
+Wire Wire Line
+	14450 7750 14750 7750
+Connection ~ 14450 7750
+$Comp
+L GND #PWR039
+U 1 1 570101A7
+P 14450 7950
+F 0 "#PWR039" H 14540 7930 30  0001 C CNN
+F 1 "GND" H 14450 7870 30  0001 C CNN
+F 2 "" H 14450 7950 60  0000 C CNN
+F 3 "" H 14450 7950 60  0000 C CNN
+	1    14450 7950
+	1    0    0    -1
+$EndComp
 $EndSCHEMATC

Commit message: Now everything is ok. + Add library by the library Wizard. + Found needed in KiCad github.
Parts:
- C1, C10, C11, C2, C3, C4, C5, C6, C7, C8, C9: footprint Capacitors_SMD:C_0603_HandSoldering -> Capacitors:CAP_0603
- DA1: footprint (none) -> TO_SOT_Packages_SMD:SOT-223
- DD1: footprint Housings_QFP:LQFP-48_7x7mm_Pitch0.5mm -> LQFP_TQFP:LQFP48
- R1, R2, R3, R4, R5: footprint Resistors_SMD:R_0603_HandSoldering -> Resistors:RES_0603
Changed lines of the file:
@@
 F 0 "R5" V 13780 2450 50  0000 C CNN
 F 1 "10k" V 13700 2600 50  0000 C CNN
-F 2 "Resistors_SMD:R_0603_HandSoldering" V 13780 2700 28  0000 C CNN
+F 2 "Resistors:RES_0603" V 13780 2700 28  0000 C CNN
 F 3 "" H 13700 2600 60  0000 C CNN
 	1    13700 2600
@@
 F 0 "C1" H 2050 4300 50  0000 L CNN
 F 1 "0.1u" H 2050 4500 50  0000 L CNN
-F 2 "Capacitors_SMD:C_0603_HandSoldering" V 2250 4250 28  0000 C BNN
+F 2 "Capacitors:CAP_0603" V 2250 4250 28  0000 C BNN
 F 3 "" H 2150 4400 60  0000 C CNN
 	1    2150 4400
@@
 F 0 "R2" V 13730 3450 50  0000 C CNN
 F 1 "10k" V 13650 3600 50  0000 C CNN
-F 2 "Resistors_SMD:R_0603_HandSoldering" V 13730 3700 28  0000 C CNN
+F 2 "Resistors:RES_0603" V 13730 3700 28  0000 C CNN
 F 3 "" H 13650 3600 60  0000 C CNN
 	1    13650 3600
@@
 F 0 "R3" V 13730 4350 50  0000 C CNN
 F 1 "10k" V 13650 4500 50  0000 C CNN
-F 2 "Resistors_SMD:R_0603_HandSoldering" V 13730 4600 28  0000 C CNN
+F 2 "Resistors:RES_0603" V 13730 4600 28  0000 C CNN
 F 3 "" H 13650 4500 60  0000 C CNN
 	1    13650 4500
@@
 F 0 "R4" V 13730 5350 50  0000 C CNN
 F 1 "10k" V 13650 5500 50  0000 C CNN
-F 2 "Resistors_SMD:R_0603_HandSoldering" V 13730 5600 28  0000 C CNN
+F 2 "Resistors:RES_0603" V 13730 5600 28  0000 C CNN
 F 3 "" H 13650 5500 60  0000 C CNN
 	1    13650 5500
@@
 F 0 "C7" H 7050 6000 50  0000 L CNN
 F 1 "1u" H 7050 6200 50  0000 L CNN
-F 2 "Capacitors_SMD:C_0603_HandSoldering" V 7250 5950 28  0000 C BNN
+F 2 "Capacitors:CAP_0603" V 7250 5950 28  0000 C BNN
 F 3 "" H 7150 6100 60  0000 C CNN
 	1    7150 6100
@@
 F 0 "C6" H 6800 6000 50  0000 L CNN
 F 1 "0.1u" H 6800 6200 50  0000 L CNN
-F 2 "Capacitors_SMD:C_0603_HandSoldering" V 7000 5950 28  0000 C BNN
+F 2 "Capacitors:CAP_0603" V 7000 5950 28  0000 C BNN
 F 3 "" H 6900 6100 60  0000 C CNN
 	1    6900 6100
@@
 F 0 "C5" H 6550 6000 50  0000 L CNN
 F 1 "0.1u" H 6550 6200 50  0000 L CNN
-F 2 "Capacitors_SMD:C_0603_HandSoldering" V 6750 5950 28  0000 C BNN
+F 2 "Capacitors:CAP_0603" V 6750 5950 28  0000 C BNN
 F 3 "" H 6650 6100 60  0000 C CNN
 	1    6650 6100
@@
 F 0 "C4" H 6300 6000 50  0000 L CNN
 F 1 "0.1u" H 6300 6200 50  0000 L CNN
-F 2 "Capacitors_SMD:C_0603_HandSoldering" V 6500 5950 28  0000 C BNN
+F 2 "Capacitors:CAP_0603" V 6500 5950 28  0000 C BNN
 F 3 "" H 6400 6100 60  0000 C CNN
 	1    6400 6100
@@
 F 0 "C3" H 6050 6000 50  0000 L CNN
 F 1 "0.1u" H 6050 6200 50  0000 L CNN
-F 2 "Capacitors_SMD:C_0603_HandSoldering" V 6250 5950 28  0000 C BNN
+F 2 "Capacitors:CAP_0603" V 6250 5950 28  0000 C BNN
 F 3 "" H 6150 6100 60  0000 C CNN
 	1    6150 6100
@@
 F 0 "C2" H 5800 6000 50  0000 L CNN
 F 1 "4u7" H 5800 6200 50  0000 L CNN
-F 2 "Capacitors_SMD:C_0603_HandSoldering" V 6000 5950 28  0000 C BNN
+F 2 "Capacitors:CAP_0603" V 6000 5950 28  0000 C BNN
 F 3 "" H 5900 6100 60  0000 C CNN
 	1    5900 6100
@@
 F 0 "C8" H 10150 5950 50  0000 L CNN
 F 1 "8p" H 10150 6150 50  0000 L CNN
-F 2 "Capacitors_SMD:C_0603_HandSoldering" V 10350 5900 28  0000 C BNN
+F 2 "Capacitors:CAP_0603" V 10350 5900 28  0000 C BNN
 F 3 "" H 10250 6050 60  0000 C CNN
 	1    10250 6050
@@
 F 0 "C9" H 10650 5950 50  0000 L CNN
 F 1 "8p" H 10650 6150 50  0000 L CNN
-F 2 "Capacitors_SMD:C_0603_HandSoldering" V 10850 5900 28  0000 C BNN
+F 2 "Capacitors:CAP_0603" V 10850 5900 28  0000 C BNN
 F 3 "" H 10750 6050 60  0000 C CNN
 	1    10750 6050
@@
 F 0 "R1" V 13680 1150 50  0000 C CNN
 F 1 "1k" V 13600 1300 50  0000 C CNN
-F 2 "Resistors_SMD:R_0603_HandSoldering" V 13680 1400 28  0000 C CNN
+F 2 "Resistors:RES_0603" V 13680 1400 28  0000 C CNN
 F 3 "" H 13600 1300 60  0000 C CNN
 	1    13600 1300
@@
 F 0 "DD1" H 7900 6000 60  0000 C CNN
 F 1 "STM32F100C8(B)" H 8550 6000 60  0000 C CNN
-F 2 "Housings_QFP:LQFP-48_7x7mm_Pitch0.5mm" H 8650 4650 60  0001 C CNN
+F 2 "LQFP_TQFP:LQFP48" H 8650 4650 60  0001 C CNN
 F 3 "" H 8650 4650 60  0000 C CNN
 	1    8650 4650
@@
 F 0 "C11" H 3950 1350 50  0000 L CNN
 F 1 "0.1u" H 3950 1550 50  0000 L CNN
-F 2 "Capacitors_SMD:C_0603_HandSoldering" V 4150 1300 28  0000 C BNN
+F 2 "Capacitors:CAP_0603" V 4150 1300 28  0000 C BNN
 F 3 "" H 4050 1450 60  0000 C CNN
 	1    4050 1450
@@
 F 0 "C10" H 2650 1350 50  0000 L CNN
 F 1 "4u7" H 2650 1550 50  0000 L CNN
-F 2 "Capacitors_SMD:C_0603_HandSoldering" V 2850 1300 28  0000 C BNN
+F 2 "Capacitors:CAP_0603" V 2850 1300 28  0000 C BNN
 F 3 "" H 2750 1450 60  0000 C CNN
 	1    2750 1450
@@
 F 0 "DA1" H 3150 1500 60  0000 C CNN
 F 1 "LD1117" H 3250 1400 60  0000 C CNN
-F 2 "" H 3250 1200 60  0001 C CNN
+F 2 "TO_SOT_Packages_SMD:SOT-223" H 3250 1200 60  0001 C CNN
 F 3 "" H 3250 1200 60  0000 C CNN
 	1    3250 1200
