File: aqua-flower_hw/aqua-flower.sch (KiCad schematic (older format))
At the start: 38 parts, among them Q1 NPN, Q2 IRLML6302, Q5 IRLML6302, SW1 BUTTON, SW2 BUTTON, SW3 BUTTON, SW4 BUTTON, SW5 BUTTON, SW6 BUTTON

Commit message: Add eeprom
Parts:
- removed XL5, XL6, XL7: CONN_3, Connect:BARREL_JACK, symbol CONN_3
- added C12: C, Capacitors:CAP_0603, symbol C
- added DA2: EEPROM_SPI, SO_DIL_TSSOP:SO8, symbol EEPROM_SPI
- added XL5, XL6, XL7: BARREL_SOCKET, Connectors:Barrel, symbol BARREL_SOCKET
- SW1, SW2, SW3, SW4, SW5, SW6: footprint Buttons_Switches_ThroughHole:SW_PUSH_SMALL -> BtnsSwitches:PUSH_THRHOLE_3-1825910-5
- XL2: footprint Socket_Strips:Socket_Strip_Straight_1x08 -> Display:84x48_LCD_Module
Connections:
- net labels added: EE_CS, EE_HOLD, EE_MISO, EE_MOSI, EE_SCK, EE_WP
- wire segments 141 -> 157
- no-connect marks 16 -> 10
Changed lines of the file:
@@
 LIBS:Tittar_kl
 LIBS:Transistors_kl
+LIBS:memory
 LIBS:aqua-flower-cache
 EELAYER 25 0
@@
 Connection ~ 13700 2900
 Connection ~ 13700 2300
-Wire Wire Line
-	14950 2400 14950 2900
 $Comp
 L GND #PWR01
 U 1 1 56EC14DF
-P 14950 2900
-F 0 "#PWR01" H 15040 2880 30  0001 C CNN
-F 1 "GND" H 14950 2820 30  0001 C CNN
-F 2 "" H 14950 2900 60  0000 C CNN
-F 3 "" H 14950 2900 60  0000 C CNN
-	1    14950 2900
+P 15400 2900
+F 0 "#PWR01" H 15490 2880 30  0001 C CNN
+F 1 "GND" H 15400 2820 30  0001 C CNN
+F 2 "" H 15400 2900 60  0000 C CNN
+F 3 "" H 15400 2900 60  0000 C CNN
+	1    15400 2900
 	1    0    0    -1
 $EndComp
@@
 F 0 "XL2" V 1100 3950 50  0000 C CNN
 F 1 "CONN_8" V 1200 3950 50  0000 C CNN
-F 2 "Socket_Strips:Socket_Strip_Straight_1x08" H 1150 3950 60  0001 C CNN
+F 2 "Display:84x48_LCD_Module" H 1150 3950 60  0001 C CNN
 F 3 "" H 1150 3950 60  0000 C CNN
 	1    1150 3950
@@
 Connection ~ 13650 3900
 Connection ~ 13650 3300
-Wire Wire Line
-	14950 3400 14950 3900
 $Comp
 L GND #PWR06
 U 1 1 56EC30E1
-P 14950 3900
-F 0 "#PWR06" H 15040 3880 30  0001 C CNN
-F 1 "GND" H 14950 3820 30  0001 C CNN
-F 2 "" H 14950 3900 60  0000 C CNN
-F 3 "" H 14950 3900 60  0000 C CNN
-	1    14950 3900
+P 15400 3900
+F 0 "#PWR06" H 15490 3880 30  0001 C CNN
+F 1 "GND" H 15400 3820 30  0001 C CNN
+F 2 "" H 15400 3900 60  0000 C CNN
+F 3 "" H 15400 3900 60  0000 C CNN
+	1    15400 3900
 	1    0    0    -1
 $EndComp
@@
 F 0 "SW1" H 6450 9250 50  0000 C CNN
 F 1 "BUTTON" H 6750 9250 50  0000 C CNN
-F 2 "Buttons_Switches_ThroughHole:SW_PUSH_SMALL" H 6650 9100 60  0001 C CNN
+F 2 "BtnsSwitches:PUSH_THRHOLE_3-1825910-5" H 6650 9100 60  0001 C CNN
 F 3 "" H 6650 9100 60  0000 C CNN
 	1    6650 9100
@@
 F 0 "SW2" H 7200 8850 50  0000 C CNN
 F 1 "BUTTON" H 7500 8850 50  0000 C CNN
-F 2 "Buttons_Switches_ThroughHole:SW_PUSH_SMALL" H 7400 8700 60  0001 C CNN
+F 2 "BtnsSwitches:PUSH_THRHOLE_3-1825910-5" H 7400 8700 60  0001 C CNN
 F 3 "" H 7400 8700 60  0000 C CNN
 	1    7400 8700
@@
 F 0 "SW3" H 7250 9650 50  0000 C CNN
 F 1 "BUTTON" H 7550 9650 50  0000 C CNN
-F 2 "Buttons_Switches_ThroughHole:SW_PUSH_SMALL" H 7450 9500 60  0001 C CNN
+F 2 "BtnsSwitches:PUSH_THRHOLE_3-1825910-5" H 7450 9500 60  0001 C CNN
 F 3 "" H 7450 9500 60  0000 C CNN
 	1    7450 9500
@@
 F 0 "SW4" H 7850 9250 50  0000 C CNN
 F 1 "BUTTON" H 8150 9250 50  0000 C CNN
-F 2 "Buttons_Switches_ThroughHole:SW_PUSH_SMALL" H 8050 9100 60  0001 C CNN
+F 2 "BtnsSwitches:PUSH_THRHOLE_3-1825910-5" H 8050 9100 60  0001 C CNN
 F 3 "" H 8050 9100 60  0000 C CNN
 	1    8050 9100
@@
 F 0 "SW5" H 9550 8850 50  0000 C CNN
 F 1 "BUTTON" H 9850 8850 50  0000 C CNN
-F 2 "Buttons_Switches_ThroughHole:SW_PUSH_SMALL" H 9750 8700 60  0001 C CNN
+F 2 "BtnsSwitches:PUSH_THRHOLE_3-1825910-5" H 9750 8700 60  0001 C CNN
 F 3 "" H 9750 8700 60  0000 C CNN
 	1    9750 8700
@@
 F 0 "SW6" H 9550 9200 50  0000 C CNN
 F 1 "BUTTON" H 9850 9200 50  0000 C CNN
-F 2 "Buttons_Switches_ThroughHole:SW_PUSH_SMALL" H 9750 9050 60  0001 C CNN
+F 2 "BtnsSwitches:PUSH_THRHOLE_3-1825910-5" H 9750 9050 60  0001 C CNN
 F 3 "" H 9750 9050 60  0000 C CNN
 	1    9750 9050
@@
 Wire Wire Line
 	7200 4450 7400 4450
-NoConn ~ 7400 4050
-NoConn ~ 7400 4150
-NoConn ~ 7400 4250
-NoConn ~ 7400 4350
 $Comp
 L +12V #PWR026
@@
 $EndComp
 Wire Wire Line
-	1300 1150 1700 1150
+	1200 1150 1700 1150
 $Comp
 L GND #PWR027
 U 1 1 56FF79C6
-P 1750 1500
-F 0 "#PWR027" H 1840 1480 30  0001 C CNN
-F 1 "GND" H 1750 1420 30  0001 C CNN
-F 2 "" H 1750 1500 60  0000 C CNN
-F 3 "" H 1750 1500 60  0000 C CNN
-	1    1750 1500
-	1    0    0    -1
-$EndComp
-NoConn ~ 1300 1350
+P 1150 2000
+F 0 "#PWR027" H 1240 1980 30  0001 C CNN
+F 1 "GND" H 1150 1920 30  0001 C CNN
+F 2 "" H 1150 2000 60  0000 C CNN
+F 3 "" H 1150 2000 60  0000 C CNN
+	1    1150 2000
+	1    0    0    -1
+$EndComp
+NoConn ~ 1200 1350
 Wire Wire Line
 	2600 1150 2950 1150
@@
 	-1   0    0    1
 $EndComp
-$Comp
-L CONN_3 XL5
-U 1 1 570022F0
-P 1100 1250
-F 0 "XL5" V 1050 1250 40  0000 C CNN
-F 1 "CONN_3" V 1150 1250 40  0000 C CNN
-F 2 "Connect:BARREL_JACK" H 1100 1250 60  0001 C CNN
-F 3 "" H 1100 1250 60  0000 C CNN
-	1    1100 1250
-	1    0    0    -1
-$EndComp
-Wire Wire Line
-	1300 1250 1750 1250
-Wire Wire Line
-	1750 1250 1750 1500
-$Comp
-L CONN_3 XL6
-U 1 1 570033E6
-P 15300 2400
-F 0 "XL6" V 15250 2400 40  0000 C CNN
-F 1 "CONN_3" V 15350 2400 40  0000 C CNN
-F 2 "Connect:BARREL_JACK" H 15300 2400 60  0001 C CNN
-F 3 "" H 15300 2400 60  0000 C CNN
-	1    15300 2400
-	-1   0    0    -1
-$EndComp
-$Comp
-L CONN_3 XL7
-U 1 1 57003936
-P 15300 3400
-F 0 "XL7" V 15250 3400 40  0000 C CNN
-F 1 "CONN_3" V 15350 3400 40  0000 C CNN
-F 2 "Connect:BARREL_JACK" H 15300 3400 60  0001 C CNN
-F 3 "" H 15300 3400 60  0000 C CNN
-	1    15300 3400
-	-1   0    0    -1
-$EndComp
-Wire Wire Line
-	14950 2400 15100 2400
-Wire Wire Line
-	14950 3400 15100 3400
+Wire Wire Line
+	1150 1750 1150 2000
 $Comp
 L PWR_FLAG #FLG033
@@
 L PWR_FLAG #FLG034
 U 1 1 57009282
-P 1500 1350
-F 0 "#FLG034" H 1500 1620 30  0001 C CNN
-F 1 "PWR_FLAG" H 1500 1550 30  0000 C CNN
-F 2 "" H 1500 1350 60  0000 C CNN
-F 3 "" H 1500 1350 60  0000 C CNN
-	1    1500 1350
+P 900 1850
+F 0 "#FLG034" H 900 2120 30  0001 C CNN
+F 1 "PWR_FLAG" H 900 2050 30  0000 C CNN
+F 2 "" H 900 1850 60  0000 C CNN
+F 3 "" H 900 1850 60  0000 C CNN
+	1    900  1850
 	-1   0    0    1
 $EndComp
 Wire Wire Line
-	1500 1350 1500 1250
-Connection ~ 1500 1250
-Wire Wire Line
-	14500 2300 15100 2300
+	900  1650 900  1850
+Connection ~ 900  1750
 Wire Wire Line
 	14450 3300 15100 3300
@@
 	1    0    0    -1
 $EndComp
-NoConn ~ 9900 3650
-NoConn ~ 9900 3750
+$Comp
+L EEPROM_SPI DA2
+U 1 1 56FE44F0
+P 6150 1350
+F 0 "DA2" H 6350 1750 60  0000 C CNN
+F 1 "EEPROM_SPI" H 5850 1750 60  0000 C CNN
+F 2 "SO_DIL_TSSOP:SO8" H 6150 1350 60  0001 C CNN
+F 3 "" H 6150 1350 60  0000 C CNN
+	1    6150 1350
+	-1   0    0    -1
+$EndComp
+$Comp
+L C C12
+U 1 1 56FE47E0
+P 5400 1500
+F 0 "C12" H 5300 1400 50  0000 L CNN
+F 1 "C" H 5300 1600 50  0000 L CNN
+F 2 "Capacitors:CAP_0603" V 5500 1350 28  0000 C BNN
+F 3 "" H 5400 1500 60  0000 C CNN
+	1    5400 1500
+	1    0    0    -1
+$EndComp
+Wire Wire Line
+	5300 1150 5750 1150
+Wire Wire Line
+	5400 1150 5400 1300
+Connection ~ 5400 1150
+Wire Wire Line
+	5750 1250 5650 1250
+Wire Wire Line
+	5750 1350 5650 1350
+Wire Wire Line
+	5750 1450 5650 1450
+Wire Wire Line
+	5650 1450 5650 2000
+Wire Wire Line
+	5400 1700 5400 1850
+Wire Wire Line
+	5400 1850 5650 1850
+Connection ~ 5650 1850
+$Comp
+L GND #PWR036
+U 1 1 56FE50A2
+P 5650 2000
+F 0 "#PWR036" H 5740 1980 30  0001 C CNN
+F 1 "GND" H 5650 1920 30  0001 C CNN
+F 2 "" H 5650 2000 60  0000 C CNN
+F 3 "" H 5650 2000 60  0000 C CNN
+	1    5650 2000
+	1    0    0    -1
+$EndComp
+$Comp
+L +3.3V #PWR037
+U 1 1 56FE5106
+P 5300 1150
+F 0 "#PWR037" H 5300 1110 30  0001 C CNN
+F 1 "+3.3V" H 5380 1180 30  0000 C CNN
+F 2 "" H 5300 1150 60  0000 C CNN
+F 3 "" H 5300 1150 60  0000 C CNN
+	1    5300 1150
+	-1   0    0    1
+$EndComp
+Text Label 5650 1250 2    60   ~ 0
+EE_HOLD
+Text Label 5650 1350 2    60   ~ 0
+EE_WP
+Wire Wire Line
+	6650 1150 6750 1150
+Wire Wire Line
+	6650 1250 6750 1250
+Wire Wire Line
+	6650 1350 6750 1350
+Wire Wire Line
+	6650 1450 6750 1450
+Text Label 6750 1150 0    60   ~ 0
+EE_CS
+Text Label 6750 1250 0    60   ~ 0
+EE_MISO
+Text Label 6750 1350 0    60   ~ 0
+EE_SCK
+Text Label 6750 1450 0    60   ~ 0
+EE_MOSI
+Wire Wire Line
+	9900 3650 10100 3650
+Wire Wire Line
+	9900 3750 10100 3750
+Text Label 10100 3650 0    60   ~ 0
+EE_HOLD
+Text Label 10100 3750 0    60   ~ 0
+EE_WP
+Wire Wire Line
+	7400 4050 7200 4050
+Wire Wire Line
+	7400 4150 7200 4150
+Wire Wire Line
+	7400 4250 7200 4250
+Wire Wire Line
+	7400 4350 7200 4350
+Text Label 7200 4050 2    60   ~ 0
+EE_CS
+Text Label 7200 4150 2    60   ~ 0
+EE_MISO
+Text Label 7200 4250 2    60   ~ 0
+EE_MOSI
+Text Label 7200 4350 2    60   ~ 0
+EE_SCK
+$Comp
+L BARREL_SOCKET XL5
+U 1 1 56FE8497
+P 1000 1250
+F 0 "XL5" H 850 1500 60  0000 C CNN
+F 1 "BARREL_SOCKET" V 700 1250 60  0000 C CNN
+F 2 "Connectors:Barrel" H 1000 1250 60  0001 C CNN
+F 3 "" H 1000 1250 60  0000 C CNN
+	1    1000 1250
+	1    0    0    -1
+$EndComp
+Wire Wire Line
+	900  1750 1150 1750
+$Comp
+L BARREL_SOCKET XL6
+U 1 1 56FE9BE8
+P 15300 2400
+F 0 "XL6" H 15150 2650 60  0000 C CNN
+F 1 "BARREL_SOCKET" V 15000 2400 60  0000 C CNN
+F 2 "Connectors:Barrel" H 15300 2400 60  0001 C CNN
+F 3 "" H 15300 2400 60  0000 C CNN
+	1    15300 2400
+	-1   0    0    -1
+$EndComp
+Wire Wire Line
+	15400 2900 15400 2800
+$Comp
+L BARREL_SOCKET XL7
+U 1 1 56FEA65A
+P 15300 3400
+F 0 "XL7" H 15150 3650 60  0000 C CNN
+F 1 "BARREL_SOCKET" V 15000 3400 60  0000 C CNN
+F 2 "Connectors:Barrel" H 15300 3400 60  0001 C CNN
+F 3 "" H 15300 3400 60  0000 C CNN
+	1    15300 3400
+	-1   0    0    -1
+$EndComp
+Wire Wire Line
+	15400 3900 15400 3800
+Wire Wire Line
+	14500 2300 15100 2300
 $EndSCHEMATC

Commit message: Replace straight pin connectors
Parts:
- XL1: footprint Socket_Strips:Socket_Strip_Straight_1x05 -> Connectors:PLS-5
- XL3: footprint Socket_Strips:Socket_Strip_Straight_1x03 -> Connectors:PLS-3
- XL4: footprint Socket_Strips:Socket_Strip_Straight_1x04 -> Connectors:PLS-4
Connections:
- net labels added: 12V
Changed lines of the file:
@@
 F 0 "XL4" H 1100 6300 60  0000 C CNN
 F 1 "ST_SWD" H 1450 6300 60  0000 C CNN
-F 2 "Socket_Strips:Socket_Strip_Straight_1x04" H 1250 6000 60  0001 C CNN
+F 2 "Connectors:PLS-4" H 1250 6000 60  0001 C CNN
 F 3 "" H 1250 6000 60  0000 C CNN
 	1    1250 6000
@@
 F 0 "XL3" V 1150 7250 40  0000 C CNN
 F 1 "CONN_3" V 1250 7250 40  0000 C CNN
-F 2 "Socket_Strips:Socket_Strip_Straight_1x03" H 1200 7250 60  0001 C CNN
+F 2 "Connectors:PLS-3" H 1200 7250 60  0001 C CNN
 F 3 "" H 1200 7250 60  0000 C CNN
 	1    1200 7250
@@
 F 0 "XL1" V 1100 2850 50  0000 C CNN
 F 1 "CONN_5" V 1200 2850 50  0000 C CNN
-F 2 "Socket_Strips:Socket_Strip_Straight_1x05" H 1150 2850 60  0001 C CNN
+F 2 "Connectors:PLS-5" H 1150 2850 60  0001 C CNN
 F 3 "" H 1150 2850 60  0000 C CNN
 	1    1150 2850
@@
 Wire Wire Line
 	14500 2300 15100 2300
+Text Label 14750 2300 0    60   ~ 0
+12V
+Text Label 14750 3300 0    60   ~ 0
+12V
 $EndSCHEMATC

Commit message: PCB finalize. Ready to production.
Parts:
- removed XL1: CONN_5, Connectors:PLS-5, symbol CONN_5
- added XL1: CONN_6, Connectors:PLS-6, symbol CONN_6
- C10: value 4u7 -> 10u; footprint Capacitors:CAP_0603 -> Capacitors:CAP_0805
- C12: value C -> 0.1u
Connections:
- net labels added: PUMP1, PUMP2
- net labels removed: 12V
- wire segments 157 -> 159
Changed lines of the file:
@@
 EESchema Schematic File Version 2
-LIBS:aqua-flower-rescue
 LIBS:Connectors_kl
 LIBS:display_kl
@@
 LIBS:Transistors_kl
 LIBS:memory
-LIBS:aqua-flower-cache
 EELAYER 25 0
 EELAYER END
@@
 Text Label 10100 4150 0    60   ~ 0
 CC_MOSI
-$Comp
-L CONN_5 XL1
-U 1 1 56FE3EA4
-P 1150 2850
-F 0 "XL1" V 1100 2850 50  0000 C CNN
-F 1 "CONN_5" V 1200 2850 50  0000 C CNN
-F 2 "Connectors:PLS-5" H 1150 2850 60  0001 C CNN
-F 3 "" H 1150 2850 60  0000 C CNN
-	1    1150 2850
-	-1   0    0    -1
-$EndComp
 Wire Wire Line
 	1350 2650 1550 2650
@@
 Wire Wire Line
 	1350 3050 1550 3050
+Text Label 1550 2950 0    60   ~ 0
+CC_SCK
+Text Label 1550 3050 0    60   ~ 0
+CC_CS
+Text Label 1550 2850 0    60   ~ 0
+CC_MISO
 Text Label 1550 2750 0    60   ~ 0
-CC_SCK
-Text Label 1550 2850 0    60   ~ 0
-CC_CS
-Text Label 1550 2950 0    60   ~ 0
-CC_MISO
-Text Label 1550 3050 0    60   ~ 0
 CC_MOSI
 $Comp
@@
 P 2750 1450
 F 0 "C10" H 2650 1350 50  0000 L CNN
-F 1 "4u7" H 2650 1550 50  0000 L CNN
-F 2 "Capacitors:CAP_0603" V 2850 1300 28  0000 C BNN
+F 1 "10u" H 2650 1550 50  0000 L CNN
+F 2 "Capacitors:CAP_0805" V 2850 1300 28  0000 C BNN
 F 3 "" H 2750 1450 60  0000 C CNN
 	1    2750 1450
@@
 P 5400 1500
 F 0 "C12" H 5300 1400 50  0000 L CNN
-F 1 "C" H 5300 1600 50  0000 L CNN
+F 1 "0.1u" H 5300 1600 50  0000 L CNN
 F 2 "Capacitors:CAP_0603" V 5500 1350 28  0000 C BNN
 F 3 "" H 5400 1500 60  0000 C CNN
@@
 	14500 2300 15100 2300
 Text Label 14750 2300 0    60   ~ 0
-12V
+PUMP1
 Text Label 14750 3300 0    60   ~ 0
-12V
+PUMP2
+$Comp
+L CONN_6 XL1
+U 1 1 5701903C
+P 1150 2900
+F 0 "XL1" V 1100 2900 50  0000 C CNN
+F 1 "CONN_6" V 1200 2900 50  0000 C CNN
+F 2 "Connectors:PLS-6" H 1150 2900 60  0001 C CNN
+F 3 "" H 1150 2900 60  0000 C CNN
+	1    1150 2900
+	-1   0    0    -1
+$EndComp
+Wire Wire Line
+	1350 3150 1550 3150
+Wire Wire Line
+	1550 3150 1550 3300
+$Comp
+L GND #PWR038
+U 1 1 57019388
+P 1550 3300
+F 0 "#PWR038" H 1640 3280 30  0001 C CNN
+F 1 "GND" H 1550 3220 30  0001 C CNN
+F 2 "" H 1550 3300 60  0000 C CNN
+F 3 "" H 1550 3300 60  0000 C CNN
+	1    1550 3300
+	1    0    0    -1
+$EndComp
 $EndSCHEMATC

Commit message: Update sch of pcb
Parts:
- added Q3, Q4: NPN, symbol NPN
Connections:
- wire segments 159 -> 163
