File: aqua-flower_hw/aqua-flower.kicad_pcb (KiCad board)
At the start: 2 copper layers, 84 x 45 mm, 40 parts, among them Q1 NPN, Q2 IRLML6302, Q5 IRLML6302, SW1 BUTTON, SW2 BUTTON, SW3 BUTTON, SW4 BUTTON, SW5 BUTTON, SW6 BUTTON

Commit message: Fix silk
Other:
- board text added: "T"
Changed lines of the file:
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@@
     (links 113)
     (no_connects 0)
-    (area 98.924999 92.924999 183.075001 138.075001)
+    (area 95.124999 78.15 196 141.875001)
     (thickness 1.5)
-    (drawings 7)
+    (drawings 8)
     (tracks 1343)
     (zones 0)
@@
     (visible_elements 7FFFF7FF)
     (pcbplotparams
-      (layerselection 0x00030_80000001)
-      (usegerberextensions false)
+      (layerselection 0x010e0_80000001)
+      (usegerberextensions true)
       (excludeedgelayer true)
       (linewidth 0.100000)
@@
       (outputformat 1)
       (mirror false)
-      (drillshape 1)
+      (drillshape 0)
       (scaleselection 1)
-      (outputdirectory ""))
+      (outputdirectory gerber/))
   )
   (net 0 "")
@@
     (at 129.3 104.7)
     (attr smd)
-    (fp_text reference C7 (at 2.2 0.4) (layer F.SilkS)
-      (effects (font (size 0.6 0.6) (thickness 0.15)))
-    )
-    (fp_text value 1u (at 2.2 -0.4) (layer F.SilkS)
+    (fp_text reference C7 (at -1.2 1.4) (layer F.SilkS)
+      (effects (font (size 0.6 0.6) (thickness 0.15)))
+    )
+    (fp_text value 1u (at 0.9 1.3) (layer F.SilkS)
       (effects (font (size 0.6 0.6) (thickness 0.15)))
     )
@@
     (at 132.3 104.7 180)
     (attr smd)
-    (fp_text reference C8 (at 2.2 0.4 180) (layer F.SilkS)
-      (effects (font (size 0.6 0.6) (thickness 0.15)))
-    )
-    (fp_text value 8p (at 2.2 -0.5 180) (layer F.SilkS)
+    (fp_text reference C8 (at -2.2 -0.9 180) (layer F.SilkS)
+      (effects (font (size 0.6 0.6) (thickness 0.15)))
+    )
+    (fp_text value 8p (at -1 -1.4 180) (layer F.SilkS)
       (effects (font (size 0.6 0.6) (thickness 0.15)))
     )
@@
   (module LQFP_TQFP:LQFP48 (layer F.Cu)
     (at 134.2 114.1 270)
-    (fp_text reference DD1 (at 0.39878 -2.49936 270) (layer F.SilkS)
+    (fp_text reference DD1 (at 1.4 0.1 360) (layer F.SilkS)
       (effects (font (size 0.59944 0.59944) (thickness 0.14986)))
     )
-    (fp_text value "STM32F100C8(B)" (at -1.80086 0.09906 270) (layer F.SilkS)
+    (fp_text value "STM32F100C8(B)" (at -5.8 -0.3 360) (layer F.SilkS)
       (effects (font (size 0.59944 0.59944) (thickness 0.14986)))
     )
@@
   (module Display:84x48_LCD_Module (layer F.Cu)
     (at 132 94)
-    (fp_text reference XL2 (at 0 21.59) (layer F.SilkS)
+    (fp_text reference XL2 (at 2.2 20.2) (layer F.SilkS)
       (effects (font (size 1 1) (thickness 0.15)))
     )
@@
       (net 3 GND))
   )
+  (gr_text T (at 157.3 95.3) (layer F.SilkS)
+    (effects (font (size 1.5 1.5) (thickness 0.3)))
+  )
   (gr_text "Aqua Flower v.1" (at 167.8 135.9) (layer F.SilkS)
